Commit message: Full codes added

File: Franka-LHT-Simulator/Objects/YcbMustardBottle/model.urdf (robot description, URDF)
Before this commit: robot model.urdf, 1 links, 0 joints
Links:
- link baseLink: geometry collision mesh filename=collision_vhacd.obj scale=1 1 0.6; visual mesh filename=textured_simple_reoriented.obj scale=1 1 1

File: Franka-LHT-Simulator/Objects/plastic_water_bottle/urdf/plastic_water_bottle.urdf (robot description, URDF)
Before this commit: robot plastic_water_bottle, 2 links, 1 joints
Links:
- link link1: geometry visual mesh filename=package://plastic_water_bottle/meshes/link1.STL

File: Franka-LHT-Simulator/Objects/wooden_crate/wooden_crate.urdf (robot description, URDF)
Before this commit: robot bottle, 1 links, 0 joints
Links:
- link base_link: geometry collision mesh filename=meshes/decomp.obj scale=0.01 0.01 0.0000006; visual mesh filename=meshes/wooden_bottle_crate.obj scale=0.01 0.01 0.01

File: frankaKitchenPybullet/kitchen_assets/item_assets/kettle.urdf (robot description, URDF)
Before this commit: robot kettle_urdf, 2 links, 1 joints
Links:
- link kettleroot_1: geometry collision box size=0.244 0.244 0.116; collision cylinder length=0.1 radius=0.031
